File: eagle/controller2.brd (EAGLE design)
At the start: 77.1 x 48.2 mm, 18 parts, among them K1 SRD-05VDC-SL-C, K2 SRD-05VDC-SL-C, T1 BC547, T2 BC547, X1 VCC, X2 IN1, X3 IN2

Commit message: Update to Version 1.1
Parts:
- moved HLK1 89.1 mm to (10.7, 26.7), turned to 90 degrees
- moved X1 74.9 mm to (10.7, 5.59), turned to 0 degrees
- moved U$2 56.9 mm to (79.0, 2.54)
- moved U$4 52.5 mm to (79.0, 41.4)
- moved T2 50.8 mm to (40.6, 40.1), turned to 90 degrees
- moved R2 48.7 mm to (46.2, 40.1), turned to 180 degrees
- moved T1 48.2 mm to (24.1, 40.1), turned to 90 degrees
- moved R1 46.0 mm to (29.7, 40.1), turned to 180 degrees
- moved LED2 39.8 mm to (49.3, 37.0), turned to 90 degrees
- moved U$3 39.1 mm to (2.79, 2.54)
- moved LED1 37.1 mm to (32.8, 37.0), turned to 90 degrees
- moved U$1 33.8 mm to (67.6, 22.4), turned to 180 degrees
- moved K2 28.1 mm to (46.0, 19.6)
- moved X3 26.9 mm to (42.9, 5.59)
- moved K1 24.3 mm to (29.5, 19.6)
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Connections:
- net 0V: now also X1.2; no longer X1.1
- net VCC: now also X1.1; no longer X1.2
Routing:
- net VCC: track 43.0 -> 69.3 mm
- net 0V: track 69.0 -> 45.4 mm, vias 1 -> 0
- net GND: track 83.4 -> 64.5 mm
- net N$3: track 32.2 -> 13.5 mm
- net N$1: track 32.2 -> 13.6 mm
- net +5V: track 69.3 -> 57.9 mm
- net N$14: track 25.5 -> 18.2 mm
- net N$15: track 43.6 -> 36.9 mm
- net N$2: track 13.1 -> 9.33 mm
- net N$11: track 13.1 -> 9.33 mm
- net N$8: track 2.43 -> 4.95 mm
- net N$20: track 4.34 -> 2.12 mm
- net N$9: track 3.17 -> 4.95 mm
Other:
- board size 77.1 x 48.2 mm -> 81.5 x 43.7 mm
- board text added: "2 Port UHC 1.1"
- board text added: "PWR"
- board text added: "VENT1"
- board text added: "VENT2"
- board text removed: "2 PORT UNDERFLOOR HEATING CONTROLLER 1.0"

Commit message: refactoring
Parts:
- removed R1, R2: 1k, rcl:0204/5
- moved LED2 5.16 mm to (45.2, 40.1), turned to 180 degrees
- moved LED1 5.16 mm to (28.7, 40.1), turned to 180 degrees
- moved D1 3.05 mm to (29.2, 34.8)
- moved D2 3.05 mm to (45.7, 34.8)
Connections:
- removed net N$19: LED2.K, R2.1
- removed net N$20: LED1.K, R1.1
- net N$14: now also U$1.JP1.4; no longer U$1.JP2.4
- net N$15: now also U$1.JP1.3; no longer U$1.JP2.3
- net N$8: now also LED2.K; no longer R2.2
- net N$9: now also LED1.K; no longer R1.2
Routing:
- net N$14: track 18.2 -> 41.0 mm
- net N$15: track 36.9 -> 58.2 mm
- net +5V: track 57.9 -> 69.0 mm
- net VCC: track 69.3 -> 67.1 mm
- net N$19: track 2.12 -> 0.00 mm
- net N$20: track 2.12 -> 0.00 mm
- net GND: track 64.5 -> 66.1 mm
