File: eagle/controller2.sch (EAGLE design)
At the start: 27 parts, among them K1 SRD-05VDC-SL-C, K2 SRD-05VDC-SL-C, K3 SRD-05VDC-SL-C, K4 SRD-05VDC-SL-C, T1 BC547, T2 BC547, T3 BC547, T4 BC547, X1 VCC, X2 IN1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

Commit message: Add different board version
Parts:
- removed D3, D4: 1N4001, tango:1N4001
- removed K3, K4: SRD-05VDC-SL-C, SRD-05VDC-SL-C (1):SRD-05VDC-SL-C
- removed LED3, LED4: RED, led:LED3MM
- removed R3, R4: 1k, rcl:R-EU_0204/5
- removed T3, T4: BC547, transistor:BC547
- removed X4: IN3, con-wago-500:W237-102
- removed X5: IN4, con-wago-500:W237-102
Connections:
- removed net N$10: R4.2, T4.B
- removed net N$12: K3.NO, X4-1.KL
- removed net N$13: K4.NO, X5-1.KL
- removed net N$16: LED3.A, U$1.D3
- removed net N$17: LED4.A, U$1.D4
- removed net N$18: LED3.C, R3.1
- removed net N$4: D3.ANODE, K3.A2, T3.C
- removed net N$5: D4.ANODE, K4.A2, T4.C
- removed net N$6: LED4.C, R4.1
- removed net N$7: R3.2, T3.B
- net +5V: no longer D3.CATHODE, D4.CATHODE, K3.A1, K4.A1
- net 0V: no longer X4-2.KL, X5-2.KL
- net GND: no longer T3.E, T4.E
- net VCC: no longer K3.COM, K4.COM
Other:
- moved on the sheet: LED2, R2

Commit message: Update to Version 1.1
Connections:
- net 0V: now also X1-2.KL; no longer X1-1.KL
- net VCC: now also X1-1.KL; no longer X1-2.KL
Other:
- moved on the sheet: LED2, R2, X1-1, X1-2
Changed lines of the file:
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@@
 <attribute name="NAME" x="276.86" y="44.069" size="1.778" layer="95" rot="MR180"/>
 </instance>
-<instance part="X1" gate="-1" x="73.66" y="20.32" smashed="yes">
+<instance part="X1" gate="-1" x="73.66" y="25.4" smashed="yes">
+<attribute name="NAME" x="73.66" y="26.289" size="1.778" layer="95" rot="R180"/>
+</instance>
+<instance part="X1" gate="-2" x="73.66" y="20.32" smashed="yes">
+<attribute name="VALUE" x="71.12" y="16.637" size="1.778" layer="96"/>
 <attribute name="NAME" x="73.66" y="21.209" size="1.778" layer="95" rot="R180"/>
-</instance>
-<instance part="X1" gate="-2" x="73.66" y="25.4" smashed="yes">
-<attribute name="VALUE" x="71.12" y="21.717" size="1.778" layer="96"/>
-<attribute name="NAME" x="73.66" y="26.289" size="1.778" layer="95" rot="R180"/>
 </instance>
 <instance part="GND1" gate="1" x="149.86" y="27.94" smashed="yes">
@@
 <attribute name="VALUE" x="179.07" y="72.898" size="1.778" layer="96"/>
 </instance>
-<instance part="R2" gate="G$1" x="182.88" y="58.42" smashed="yes">
-<attribute name="NAME" x="179.07" y="59.9186" size="1.778" layer="95"/>
-<attribute name="VALUE" x="179.07" y="55.118" size="1.778" layer="96"/>
+<instance part="R2" gate="G$1" x="182.88" y="55.88" smashed="yes">
+<attribute name="NAME" x="179.07" y="57.3786" size="1.778" layer="95"/>
+<attribute name="VALUE" x="179.07" y="52.578" size="1.778" layer="96"/>
 </instance>
 <instance part="LED1" gate="G$1" x="162.56" y="76.2" smashed="yes" rot="R90">
@@
 <attribute name="VALUE" x="167.132" y="81.915" size="1.778" layer="96" rot="R180"/>
 </instance>
-<instance part="LED2" gate="G$1" x="165.1" y="58.42" smashed="yes" rot="R90">
-<attribute name="NAME" x="169.672" y="61.976" size="1.778" layer="95" rot="R180"/>
-<attribute name="VALUE" x="169.672" y="64.135" size="1.778" layer="96" rot="R180"/>
+<instance part="LED2" gate="G$1" x="165.1" y="55.88" smashed="yes" rot="R90">
+<attribute name="NAME" x="169.672" y="59.436" size="1.778" layer="95" rot="R180"/>
+<attribute name="VALUE" x="169.672" y="61.595" size="1.778" layer="96" rot="R180"/>
 </instance>
 </instances>
@@
 <pinref part="HLK1" gate="G$1" pin="AC1"/>
 <wire x1="86.36" y1="25.4" x2="88.9" y2="25.4" width="0.1524" layer="91"/>
-<wire x1="86.36" y1="25.4" x2="86.36" y2="10.16" width="0.1524" layer="91"/>
+<pinref part="P+2" gate="VCC" pin="VCC"/>
+<pinref part="X1" gate="-1" pin="KL"/>
+<wire x1="78.74" y1="25.4" x2="86.36" y2="25.4" width="0.1524" layer="91"/>
 <junction x="86.36" y="25.4"/>
 <wire x1="86.36" y1="10.16" x2="248.92" y2="10.16" width="0.1524" layer="91"/>
@@
 <wire x1="238.76" y1="53.34" x2="248.92" y2="53.34" width="0.1524" layer="91"/>
 <junction x="248.92" y="53.34"/>
-<pinref part="P+2" gate="VCC" pin="VCC"/>
-<pinref part="X1" gate="-2" pin="KL"/>
-<wire x1="78.74" y1="25.4" x2="86.36" y2="25.4" width="0.1524" layer="91"/>
+<wire x1="86.36" y1="10.16" x2="86.36" y2="25.4" width="0.1524" layer="91"/>
 </segment>
 </net>
@@
 <wire x1="259.08" y1="43.18" x2="259.08" y2="7.62" width="0.1524" layer="91"/>
 <wire x1="259.08" y1="7.62" x2="83.82" y2="7.62" width="0.1524" layer="91"/>
+<pinref part="GND2" gate="1" pin="0V"/>
+<junction x="259.08" y="7.62"/>
+<pinref part="X1" gate="-2" pin="KL"/>
 <pinref part="HLK1" gate="G$1" pin="AC2"/>
+<wire x1="78.74" y1="20.32" x2="83.82" y2="20.32" width="0.1524" layer="91"/>
 <wire x1="83.82" y1="20.32" x2="88.9" y2="20.32" width="0.1524" layer="91"/>
 <wire x1="83.82" y1="7.62" x2="83.82" y2="20.32" width="0.1524" layer="91"/>
-<pinref part="GND2" gate="1" pin="0V"/>
-<junction x="259.08" y="7.62"/>
-<pinref part="X1" gate="-1" pin="KL"/>
-<wire x1="78.74" y1="20.32" x2="83.82" y2="20.32" width="0.1524" layer="91"/>
 <junction x="83.82" y="20.32"/>
 </segment>
@@
 <pinref part="R2" gate="G$1" pin="2"/>
 <pinref part="T2" gate="G$1" pin="B"/>
-<wire x1="187.96" y1="58.42" x2="205.74" y2="58.42" width="0.1524" layer="91"/>
-<wire x1="205.74" y1="58.42" x2="205.74" y2="53.34" width="0.1524" layer="91"/>
+<wire x1="187.96" y1="55.88" x2="205.74" y2="55.88" width="0.1524" layer="91"/>
+<wire x1="205.74" y1="55.88" x2="205.74" y2="53.34" width="0.1524" layer="91"/>
 </segment>
 </net>
@@
 </segment>
 </net>
-<net name="N$14" class="0">
-<segment>
-<pinref part="U$1" gate="G$1" pin="D1"/>
-<wire x1="157.48" y1="60.96" x2="127" y2="60.96" width="0.1524" layer="91"/>
-<pinref part="LED1" gate="G$1" pin="A"/>
-<wire x1="160.02" y1="76.2" x2="157.48" y2="76.2" width="0.1524" layer="91"/>
-<wire x1="157.48" y1="76.2" x2="157.48" y2="60.96" width="0.1524" layer="91"/>
-</segment>
-</net>
-<net name="N$15" class="0">
-<segment>
-<pinref part="U$1" gate="G$1" pin="D2"/>
-<wire x1="162.56" y1="58.42" x2="127" y2="58.42" width="0.1524" layer="91"/>
-<pinref part="LED2" gate="G$1" pin="A"/>
-</segment>
-</net>
 <net name="N$19" class="0">
 <segment>
 <pinref part="R2" gate="G$1" pin="1"/>
 <pinref part="LED2" gate="G$1" pin="C"/>
-<wire x1="170.18" y1="58.42" x2="177.8" y2="58.42" width="0.1524" layer="91"/>
+<wire x1="170.18" y1="55.88" x2="177.8" y2="55.88" width="0.1524" layer="91"/>
 </segment>
 </net>
@@
 </segment>
 </net>
+<net name="N$14" class="0">
+<segment>
+<pinref part="U$1" gate="G$1" pin="D2"/>
+<wire x1="127" y1="58.42" x2="157.48" y2="58.42" width="0.1524" layer="91"/>
+<wire x1="157.48" y1="58.42" x2="157.48" y2="55.88" width="0.1524" layer="91"/>
+<pinref part="LED2" gate="G$1" pin="A"/>
+<wire x1="157.48" y1="55.88" x2="162.56" y2="55.88" width="0.1524" layer="91"/>
+</segment>
+</net>
+<net name="N$15" class="0">
+<segment>
+<pinref part="U$1" gate="G$1" pin="D1"/>
+<pinref part="LED1" gate="G$1" pin="A"/>
+<wire x1="127" y1="60.96" x2="160.02" y2="60.96" width="0.1524" layer="91"/>
+<wire x1="160.02" y1="60.96" x2="160.02" y2="76.2" width="0.1524" layer="91"/>
+</segment>
+</net>

Commit message: refactoring
Parts:
- removed R1, R2: 1k, rcl:R-EU_0204/5
Connections:
- removed net N$19: LED2.C, R2.1
- removed net N$20: LED1.C, R1.1
- net N$14: now also U$1.D5; no longer U$1.D2
- net N$15: now also U$1.D0; no longer U$1.D1
- net N$8: now also LED2.C; no longer R2.2
- net N$9: now also LED1.C; no longer R1.2
Other:
- moved on the sheet: LED1, LED2, U$1
