File: eagle/controller3.brd (EAGLE design)
At the start: 97.5 x 48.2 mm, 24 parts, among them K1 SRD-05VDC-SL-C, K2 SRD-05VDC-SL-C, K3 SRD-05VDC-SL-C, T1 BC547, T2 BC547, T3 BC547, X1 VCC, X2 IN1, X3 IN2, X4 IN3

Commit message: Update to Version 1.1
Parts:
- moved HLK1 89.1 mm to (10.7, 26.7), turned to 90 degrees
- moved U$2 85.8 mm to (95.8, 2.54)
- moved X1 74.9 mm to (10.7, 5.59), turned to 0 degrees
- moved U$4 43.1 mm to (95.8, 41.4)
- moved T3 40.5 mm to (57.1, 40.1), turned to 90 degrees
- moved T2 38.7 mm to (40.6, 40.1), turned to 90 degrees
- moved R3 38.5 mm to (62.7, 40.1), turned to 180 degrees
- moved T1 37.3 mm to (24.1, 40.1), turned to 90 degrees
- moved R2 36.8 mm to (46.2, 40.1), turned to 180 degrees
- moved R1 35.2 mm to (29.7, 40.1), turned to 180 degrees
- moved LED3 29.8 mm to (65.8, 37.0), turned to 90 degrees
- moved LED2 28.3 mm to (49.3, 37.0), turned to 90 degrees
- moved LED1 27.3 mm to (32.8, 37.0), turned to 90 degrees
- moved U$3 18.8 mm to (2.79, 2.54)
- moved U$1 18.1 mm to (84.3, 22.4), turned to 180 degrees
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Connections:
- removed net N$16: LED3.A, U$1.JP2.5
- new net N$17: LED3.A, U$1.JP1.3
- net 0V: now also X1.2; no longer X1.1
- net VCC: now also X1.1; no longer X1.2
Routing:
- net +5V: track 127.5 -> 84.3 mm
- net N$17: track 0.00 -> 37.3 mm
- net VCC: track 63.3 -> 100.3 mm
- net N$16: track 28.0 -> 0.00 mm
- net GND: track 104.9 -> 82.0 mm
- net 0V: track 86.2 -> 64.9 mm, vias 1 -> 0
- net N$4: track 32.2 -> 13.5 mm
- net N$3: track 32.2 -> 13.5 mm
- net N$1: track 32.2 -> 13.6 mm
- net N$14: track 46.2 -> 35.1 mm
- net N$15: track 63.9 -> 53.7 mm
- net N$12: track 13.1 -> 9.33 mm
- net N$2: track 13.1 -> 9.33 mm
- net N$11: track 13.1 -> 9.33 mm
- net N$20: track 5.61 -> 2.12 mm
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Other:
- board size 97.5 x 48.2 mm -> 98.2 x 43.7 mm
- board text added: "3 Port UHC 1.1"
- board text added: "PWR"
- board text added: "VENT1"
- board text added: "VENT2"
- board text added: "VENT3"
- board text removed: "3 PORT UNDERFLOOR HEATING CONTROLLER 1.0"

Commit message: refactoring
Parts:
- removed R1, R2, R3: 1k, rcl:0204/5
- added D4: 1N4001, tango:DO41-10
- added K4: SRD-05VDC-SL-C, SRD-05VDC-SL-C (1):RELAY_SRD-05VDC-SL-C
- added LED4: RED, led:LED3MM
- added T4: BC547, transistor:TO92
- added X5: IN4, con-wago-500:W237-102
- moved U$2 16.8 mm to (112.5, 2.54)
- moved U$4 16.8 mm to (112.5, 41.4)
- moved U$1 16.8 mm to (101.1, 22.4)
- moved LED2 5.16 mm to (45.2, 40.1), turned to 180 degrees
- moved LED3 5.16 mm to (61.7, 40.1), turned to 180 degrees
- moved LED1 5.16 mm to (28.7, 40.1), turned to 180 degrees
- moved D1 3.05 mm to (29.2, 34.8)
- moved D2 3.05 mm to (45.7, 34.8)
- moved D3 3.05 mm to (62.2, 34.8)
Connections:
- removed net N$17: LED3.A, U$1.JP1.3
- removed net N$18: LED3.K, R3.1
- removed net N$20: LED1.K, R1.1
- new net N$13: K4.NO, X5.1
- new net N$16: LED4.A, U$1.JP1.6
- new net N$5: D4.A, K4.A2, T4.3
- new net N$6: LED4.K, T4.2
- net +5V: now also D4.C, K4.A1
- net 0V: now also X5.2
- net GND: now also T4.1
- net N$14: now also U$1.JP1.4; no longer U$1.JP2.4
- net N$15: now also U$1.JP1.3; no longer U$1.JP2.3
- net N$19: now also LED3.A, U$1.JP1.5; no longer LED2.K, R2.1
- net N$7: now also LED3.K; no longer R3.2
- net N$8: now also LED2.K; no longer R2.2
- net N$9: now also LED1.K; no longer R1.2
- net VCC: now also K4.COM
Routing:
- net N$19: track 2.12 -> 56.6 mm
- net N$14: track 35.1 -> 74.5 mm
- net N$16: track 0.00 -> 39.1 mm
- net N$15: track 53.7 -> 91.8 mm
- net N$17: track 37.3 -> 0.00 mm
- net +5V: track 84.3 -> 120.5 mm
- net 0V: track 64.9 -> 83.9 mm
- net VCC: track 100.3 -> 118.2 mm
- net GND: track 82.0 -> 99.7 mm
- net N$5: track 0.00 -> 13.6 mm
- net N$13: track 0.00 -> 9.33 mm
- net N$6: track 0.00 -> 5.21 mm
- net N$20: track 2.12 -> 0.00 mm
- net N$18: track 2.12 -> 0.00 mm
Other:
- board size 98.2 x 43.7 mm -> 115 x 43.7 mm
- board text added: "4 Port UHC 1.1"
- board text added: "VENT4"
- board text removed: "3 Port UHC 1.1"

Commit message: refactoring
Parts:
- removed D4: 1N4001, tango:DO41-10
- removed K4: SRD-05VDC-SL-C, SRD-05VDC-SL-C (1):RELAY_SRD-05VDC-SL-C
- removed LED4: RED, led:LED3MM
- removed T4: BC547, transistor:TO92
- removed X5: IN4, con-wago-500:W237-102
- moved U$2 17.5 mm to (95.0, 2.54)
- moved U$4 17.5 mm to (95.0, 41.4)
- moved U$1 17.5 mm to (83.6, 22.4)
Connections:
- removed net N$13: K4.NO, X5.1
- removed net N$16: LED4.A, U$1.JP1.6
- removed net N$5: D4.A, K4.A2, T4.3
- removed net N$6: LED4.K, T4.2
- net +5V: no longer D4.C, K4.A1
- net 0V: no longer X5.2
- net GND: no longer T4.1
- net VCC: no longer K4.COM
Routing:
- net N$16: track 39.1 -> 0.00 mm
- net VCC: track 118.2 -> 92.6 mm
- net +5V: track 120.5 -> 97.2 mm
- net 0V: track 83.9 -> 64.6 mm
- net N$19: track 56.6 -> 39.1 mm
- net N$14: track 74.5 -> 57.0 mm
- net N$15: track 91.8 -> 74.2 mm
- net GND: track 99.7 -> 82.2 mm
- net N$5: track 13.6 -> 0.00 mm
- net N$13: track 9.33 -> 0.00 mm
- net N$6: track 5.21 -> 0.00 mm
Other:
- board size 115 x 43.7 mm -> 97.5 x 43.7 mm
- board text added: "3 Port UHC 1.1"
- board text removed: "4 Port UHC 1.1"
- board text removed: "VENT4"
