File: eagle/controller3.sch (EAGLE design)
At the start: 21 parts, among them K1 SRD-05VDC-SL-C, K2 SRD-05VDC-SL-C, K3 SRD-05VDC-SL-C, T1 BC547, T2 BC547, T3 BC547, X1 VCC, X2 IN1, X3 IN2, X4 IN3

Commit message: Update to Version 1.1
Connections:
- removed net N$16: LED3.A, U$1.D3
- new net N$17: LED3.A, U$1.D0
- net 0V: now also X1-2.KL; no longer X1-1.KL
- net VCC: now also X1-1.KL; no longer X1-2.KL
Other:
- moved on the sheet: X1-1, X1-2
Changed lines of the file:
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@@
 </instance>
 <instance part="X4" gate="-2" x="276.86" y="33.02" smashed="yes" rot="MR0">
-<attribute name="VALUE" x="279.4" y="29.337" size="1.778" layer="96" rot="MR0"/>
 <attribute name="NAME" x="276.86" y="33.909" size="1.778" layer="95" rot="MR180"/>
 </instance>
-<instance part="X1" gate="-1" x="73.66" y="20.32" smashed="yes">
+<instance part="X1" gate="-1" x="73.66" y="25.4" smashed="yes">
+<attribute name="NAME" x="73.66" y="26.289" size="1.778" layer="95" rot="R180"/>
+</instance>
+<instance part="X1" gate="-2" x="73.66" y="20.32" smashed="yes">
+<attribute name="VALUE" x="71.12" y="16.637" size="1.778" layer="96"/>
 <attribute name="NAME" x="73.66" y="21.209" size="1.778" layer="95" rot="R180"/>
-</instance>
-<instance part="X1" gate="-2" x="73.66" y="25.4" smashed="yes">
-<attribute name="VALUE" x="71.12" y="21.717" size="1.778" layer="96"/>
-<attribute name="NAME" x="73.66" y="26.289" size="1.778" layer="95" rot="R180"/>
 </instance>
 <instance part="GND1" gate="1" x="149.86" y="27.94" smashed="yes">
@@
 <pinref part="HLK1" gate="G$1" pin="AC1"/>
 <wire x1="86.36" y1="25.4" x2="88.9" y2="25.4" width="0.1524" layer="91"/>
-<wire x1="86.36" y1="25.4" x2="86.36" y2="10.16" width="0.1524" layer="91"/>
+<pinref part="P+2" gate="VCC" pin="VCC"/>
+<pinref part="X1" gate="-1" pin="KL"/>
+<wire x1="78.74" y1="25.4" x2="86.36" y2="25.4" width="0.1524" layer="91"/>
 <junction x="86.36" y="25.4"/>
 <wire x1="86.36" y1="10.16" x2="248.92" y2="10.16" width="0.1524" layer="91"/>
@@
 <wire x1="238.76" y1="33.02" x2="248.92" y2="33.02" width="0.1524" layer="91"/>
 <junction x="248.92" y="33.02"/>
-<pinref part="P+2" gate="VCC" pin="VCC"/>
-<pinref part="X1" gate="-2" pin="KL"/>
-<wire x1="78.74" y1="25.4" x2="86.36" y2="25.4" width="0.1524" layer="91"/>
+<wire x1="86.36" y1="10.16" x2="86.36" y2="25.4" width="0.1524" layer="91"/>
 </segment>
 </net>
@@
 <wire x1="259.08" y1="33.02" x2="259.08" y2="7.62" width="0.1524" layer="91"/>
 <wire x1="259.08" y1="7.62" x2="83.82" y2="7.62" width="0.1524" layer="91"/>
+<pinref part="GND2" gate="1" pin="0V"/>
+<junction x="259.08" y="7.62"/>
+<pinref part="X1" gate="-2" pin="KL"/>
 <pinref part="HLK1" gate="G$1" pin="AC2"/>
+<wire x1="78.74" y1="20.32" x2="83.82" y2="20.32" width="0.1524" layer="91"/>
 <wire x1="83.82" y1="20.32" x2="88.9" y2="20.32" width="0.1524" layer="91"/>
 <wire x1="83.82" y1="7.62" x2="83.82" y2="20.32" width="0.1524" layer="91"/>
-<pinref part="GND2" gate="1" pin="0V"/>
-<junction x="259.08" y="7.62"/>
-<pinref part="X1" gate="-1" pin="KL"/>
-<wire x1="78.74" y1="20.32" x2="83.82" y2="20.32" width="0.1524" layer="91"/>
 <junction x="83.82" y="20.32"/>
 </segment>
@@
 </segment>
 </net>
-<net name="N$14" class="0">
-<segment>
-<pinref part="U$1" gate="G$1" pin="D1"/>
-<wire x1="157.48" y1="60.96" x2="127" y2="60.96" width="0.1524" layer="91"/>
-<pinref part="LED1" gate="G$1" pin="A"/>
-<wire x1="160.02" y1="76.2" x2="157.48" y2="76.2" width="0.1524" layer="91"/>
-<wire x1="157.48" y1="76.2" x2="157.48" y2="60.96" width="0.1524" layer="91"/>
-</segment>
-</net>
-<net name="N$15" class="0">
-<segment>
-<pinref part="U$1" gate="G$1" pin="D2"/>
-<wire x1="157.48" y1="58.42" x2="127" y2="58.42" width="0.1524" layer="91"/>
-<pinref part="LED2" gate="G$1" pin="A"/>
-<wire x1="162.56" y1="55.88" x2="157.48" y2="55.88" width="0.1524" layer="91"/>
-<wire x1="157.48" y1="55.88" x2="157.48" y2="58.42" width="0.1524" layer="91"/>
-</segment>
-</net>
-<net name="N$16" class="0">
-<segment>
-<pinref part="U$1" gate="G$1" pin="D3"/>
-<wire x1="127" y1="55.88" x2="154.94" y2="55.88" width="0.1524" layer="91"/>
-<wire x1="154.94" y1="55.88" x2="154.94" y2="35.56" width="0.1524" layer="91"/>
+<net name="N$17" class="0">
+<segment>
+<wire x1="86.36" y1="83.82" x2="86.36" y2="60.96" width="0.1524" layer="91"/>
+<wire x1="86.36" y1="83.82" x2="154.94" y2="83.82" width="0.1524" layer="91"/>
+<wire x1="154.94" y1="83.82" x2="154.94" y2="35.56" width="0.1524" layer="91"/>
+<pinref part="LED3" gate="G$1" pin="A"/>
 <wire x1="154.94" y1="35.56" x2="160.02" y2="35.56" width="0.1524" layer="91"/>
-<pinref part="LED3" gate="G$1" pin="A"/>
+<pinref part="U$1" gate="G$1" pin="D0"/>
+<wire x1="86.36" y1="60.96" x2="91.44" y2="60.96" width="0.1524" layer="91"/>
 </segment>
 </net>
@@
 </segment>
 </net>
+<net name="N$14" class="0">
+<segment>
+<pinref part="U$1" gate="G$1" pin="D2"/>
+<wire x1="127" y1="58.42" x2="157.48" y2="58.42" width="0.1524" layer="91"/>
+<wire x1="157.48" y1="58.42" x2="157.48" y2="55.88" width="0.1524" layer="91"/>
+<pinref part="LED2" gate="G$1" pin="A"/>
+<wire x1="157.48" y1="55.88" x2="162.56" y2="55.88" width="0.1524" layer="91"/>
+</segment>
+</net>
+<net name="N$15" class="0">
+<segment>
+<pinref part="U$1" gate="G$1" pin="D1"/>
+<pinref part="LED1" gate="G$1" pin="A"/>
+<wire x1="127" y1="60.96" x2="160.02" y2="60.96" width="0.1524" layer="91"/>
+<wire x1="160.02" y1="60.96" x2="160.02" y2="76.2" width="0.1524" layer="91"/>
+</segment>
+</net>

Commit message: refactoring
Parts:
- removed R1, R2, R3: 1k, rcl:R-EU_0204/5
- added D4: 1N4001, tango:1N4001
- added K4: SRD-05VDC-SL-C, SRD-05VDC-SL-C (1):SRD-05VDC-SL-C
- added LED4: RED, led:LED3MM
- added T4: BC547, transistor:BC547
- added X5: IN4, con-wago-500:W237-102
Connections:
- removed net N$17: LED3.A, U$1.D0
- removed net N$18: LED3.C, R3.1
- removed net N$20: LED1.C, R1.1
- new net N$13: K4.NO, X5-1.KL
- new net N$16: LED4.A, U$1.D7
- new net N$5: D4.ANODE, K4.A2, T4.C
- new net N$6: LED4.C, T4.B
- net +5V: now also D4.CATHODE, K4.A1
- net 0V: now also X5-2.KL
- net GND: now also T4.E
- net N$14: now also U$1.D5; no longer U$1.D2
- net N$15: now also U$1.D0; no longer U$1.D1
- net N$19: now also LED3.A, U$1.D6; no longer LED2.C, R2.1
- net N$7: now also LED3.C; no longer R3.2
- net N$8: now also LED2.C; no longer R2.2
- net N$9: now also LED1.C; no longer R1.2
- net VCC: now also K4.COM
Other:
- moved on the sheet: LED1, LED2, LED3, U$1

Commit message: refactoring
Parts:
- removed D4: 1N4001, tango:1N4001
- removed K4: SRD-05VDC-SL-C, SRD-05VDC-SL-C (1):SRD-05VDC-SL-C
- removed LED4: RED, led:LED3MM
- removed T4: BC547, transistor:BC547
- removed X5: IN4, con-wago-500:W237-102
Connections:
- removed net N$13: K4.NO, X5-1.KL
- removed net N$16: LED4.A, U$1.D7
- removed net N$5: D4.ANODE, K4.A2, T4.C
- removed net N$6: LED4.C, T4.B
- net +5V: no longer D4.CATHODE, K4.A1
- net 0V: no longer X5-2.KL
- net GND: no longer T4.E
- net VCC: no longer K4.COM
