File: eagle/controller4.brd (EAGLE design)
At the start: 117.8 x 48.2 mm, 30 parts, among them K1 SRD-05VDC-SL-C, K2 SRD-05VDC-SL-C, K3 SRD-05VDC-SL-C, K4 SRD-05VDC-SL-C, T1 BC547, T2 BC547, T3 BC547, T4 BC547, X1 VCC, X2 IN1, X3 IN2, X4 IN3, X5 IN4

Commit message: Update to Version 1.1
Parts:
- moved U$2 119.3 mm to (112.5, 2.54)
- moved HLK1 89.1 mm to (10.7, 26.7), turned to 90 degrees
- moved X1 74.9 mm to (10.7, 5.59), turned to 0 degrees
- moved U$4 38.9 mm to (112.5, 41.4)
- moved T1 35.9 mm to (24.1, 40.1), turned to 90 degrees
- moved T2 35.3 mm to (40.6, 40.1), turned to 90 degrees
- moved T4 35.3 mm to (73.7, 40.1), turned to 90 degrees
- moved R4 35.1 mm to (79.0, 40.1), turned to 180 degrees
- moved T3 35.1 mm to (57.1, 40.1), turned to 90 degrees
- moved R1 33.2 mm to (29.7, 40.1), turned to 180 degrees
- moved R2 32.7 mm to (46.2, 40.1), turned to 180 degrees
- moved R3 32.5 mm to (62.7, 40.1), turned to 180 degrees
- moved LED1 30.1 mm to (32.8, 37.0), turned to 90 degrees
- moved LED2 28.6 mm to (49.3, 37.0), turned to 90 degrees
- moved LED3 27.5 mm to (65.8, 37.0), turned to 90 degrees
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Connections:
- net 0V: now also X1.2; no longer X1.1
- net N$16: now also LED4.A, U$1.JP1.4; no longer LED3.A, U$1.JP2.5
- net N$17: now also LED3.A, U$1.JP1.3; no longer LED4.A, U$1.JP2.6
- net VCC: now also X1.1; no longer X1.2
Routing:
- net VCC: track 83.7 -> 130.8 mm
- net +5V: track 156.0 -> 109.6 mm
- net 0V: track 115.6 -> 84.3 mm, vias 1 -> 0
- net GND: track 125.1 -> 98.8 mm
- net N$17: track 29.7 -> 54.1 mm
- net N$4: track 32.2 -> 13.5 mm
- net N$3: track 32.2 -> 13.5 mm
- net N$5: track 32.2 -> 13.6 mm
- net N$1: track 32.2 -> 13.6 mm
- net N$14: track 65.2 -> 51.4 mm
- net N$15: track 83.0 -> 70.0 mm
- net N$16: track 47.4 -> 36.5 mm
- net N$13: track 13.1 -> 9.33 mm
- net N$12: track 13.1 -> 9.33 mm
- net N$2: track 13.1 -> 9.33 mm
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Other:
- board size 117.8 x 48.2 mm -> 115 x 43.7 mm
- board text added: "4 Port UHC 1.1"
- board text added: "PWR"
- board text added: "VENT1"
- board text added: "VENT2"
- board text added: "VENT3"
- board text added: "VENT4"
- board text removed: "4 PORT UNDERFLOOR HEATING CONTROLLER 1.0"

Commit message: refactoring
Parts:
- removed R1, R2, R3, R4: 1k, rcl:0204/5
- moved LED4 5.16 mm to (78.2, 40.1), turned to 180 degrees
- moved LED2 5.16 mm to (45.2, 40.1), turned to 180 degrees
- moved LED3 5.16 mm to (61.7, 40.1), turned to 180 degrees
- moved LED1 5.16 mm to (28.7, 40.1), turned to 180 degrees
- moved D1 3.05 mm to (29.2, 34.8)
- moved D2 3.05 mm to (45.7, 34.8)
- moved D3 3.05 mm to (62.2, 34.8)
- moved D4 3.05 mm to (78.7, 34.8)
Connections:
- removed net N$10: R4.2, T4.2
- removed net N$17: LED3.A, U$1.JP1.3
- removed net N$18: LED3.K, R3.1
- removed net N$20: LED1.K, R1.1
- net N$14: now also U$1.JP1.4; no longer U$1.JP2.4
- net N$15: now also U$1.JP1.3; no longer U$1.JP2.3
- net N$16: now also U$1.JP1.6; no longer U$1.JP1.4
- net N$19: now also LED3.A, U$1.JP1.5; no longer LED2.K, R2.1
- net N$6: now also T4.2; no longer R4.1
- net N$7: now also LED3.K; no longer R3.2
- net N$8: now also LED2.K; no longer R2.2
- net N$9: now also LED1.K; no longer R1.2
Routing:
- net N$19: track 2.12 -> 56.6 mm
- net N$17: track 54.1 -> 0.00 mm
- net N$14: track 51.4 -> 74.5 mm
- net N$15: track 70.0 -> 91.8 mm
- net VCC: track 130.8 -> 118.2 mm
- net +5V: track 109.6 -> 120.5 mm
- net N$10: track 4.70 -> 0.00 mm
- net N$6: track 2.22 -> 5.21 mm
- net N$16: track 36.5 -> 39.1 mm
- net N$20: track 2.12 -> 0.00 mm
- net N$18: track 2.12 -> 0.00 mm
- net GND: track 98.8 -> 99.7 mm

Commit message: refactoring
Parts:
- removed U$4: (no value), holes:3,0
- added C1, C2, C3, C4: (no value), rcl:E5-5
- added C10, C11, C12, C5, C6, C7, C8, C9: (no value), rcl:C025-024X044
- added IC1: PCF8574P, micro-philips:DIL16
- added OK1, OK2, OK3, OK4: PC814, optocoupler:DIL04
- added R1, R10, R11, R12, R2, R3, R4, R5, R6, R7, R8, R9: (no value), rcl:0204/5
- added X6: IN5, con-wago-500:W237-102
- added X7: IN6, con-wago-500:W237-102
- moved LED4 6.86 mm to (85.1, 40.1), turned to 0 degrees
- moved LED1 6.86 mm to (35.6, 40.1), turned to 0 degrees
- moved LED2 6.86 mm to (52.1, 40.1), turned to 0 degrees
- moved LED3 6.86 mm to (68.6, 40.1), turned to 0 degrees
Connections:
- new net N$10: C9.1, R4.2, R6.2
- new net N$17: IC1.14, U$1.JP2.3
- new net N$18: IC1.15, U$1.JP2.4
- new net N$20: C10.1, R3.2, R8.2
- new net N$21: C11.1, R10.2, R2.2
- new net N$22: C8.1, OK4.1, R1.1
- new net N$23: C11.2, R9.2, X7.1
- new net N$24: C10.2, R7.2, X6.2
- new net N$25: C9.2, R5.2, X6.1
- new net N$26: R5.1, R6.1
- new net N$27: C12.1, C12.2, R1.2, R11.2, R12.2, X7.2
- new net N$28: C7.1, OK3.1, R2.1
- new net N$29: C6.1, OK2.1, R3.1
- new net N$30: C5.1, OK1.1, R4.1
- new net N$31: R7.1, R8.1
- new net N$32: R10.1, R9.1
- new net N$33: R11.1, R12.1
- new net VDD: IC1.16
- net 0V: now also C5.2, C6.2, C7.2, C8.2, OK1.2, OK2.2, OK3.2, OK4.2
- net GND: now also C1.-, C2.-, C3.-, C4.-, IC1.8, LED1.K, LED2.K, LED3.K, LED4.K, OK1.3, OK2.3, OK3.3, OK4.3
- net N$14: now also T2.2
- net N$15: now also T1.2
- net N$16: now also T4.2
- net N$19: now also T3.2
- net N$6: now also C1.+, IC1.7, OK1.4; no longer LED4.K, T4.2
- net N$7: now also C2.+, IC1.6, OK2.4; no longer LED3.K, T3.2
- net N$8: now also C3.+, IC1.5, OK3.4; no longer LED2.K, T2.2
- net N$9: now also C4.+, IC1.4, OK4.4; no longer LED1.K, T1.2
Routing:
- net 0V: track 83.9 -> 132.7 mm, vias 0 -> 1
- net N$8: track 5.21 -> 37.8 mm
- net N$9: track 5.21 -> 34.1 mm
- net GND: track 99.7 -> 122.8 mm
- net N$6: track 5.21 -> 27.8 mm
- net N$18: track 0.00 -> 19.9 mm
- net N$7: track 5.21 -> 23.4 mm
- net N$17: track 0.00 -> 11.3 mm
- net N$16: track 39.1 -> 47.4 mm
- net N$15: track 91.8 -> 99.5 mm
- net N$19: track 56.6 -> 64.4 mm
- net N$14: track 74.5 -> 81.9 mm
Other:
- board size 115 x 43.7 mm -> 115 x 62.7 mm
