File: eagle/controller4.sch (EAGLE design)
At the start: 27 parts, among them K1 SRD-05VDC-SL-C, K2 SRD-05VDC-SL-C, K3 SRD-05VDC-SL-C, K4 SRD-05VDC-SL-C, T1 BC547, T2 BC547, T3 BC547, T4 BC547, X1 VCC, X2 IN1, X3 IN2, X4 IN3, X5 IN4

Commit message: Update to Version 1.1
Connections:
- net 0V: now also X1-2.KL; no longer X1-1.KL
- net N$16: now also LED4.A, U$1.D5; no longer LED3.A, U$1.D3
- net N$17: now also LED3.A, U$1.D0; no longer LED4.A, U$1.D4
- net VCC: now also X1-1.KL; no longer X1-2.KL
Other:
- moved on the sheet: X1-1, X1-2
Changed lines of the file:
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@@
 <attribute name="NAME" x="276.86" y="23.749" size="1.778" layer="95" rot="MR180"/>
 </instance>
-<instance part="X1" gate="-1" x="73.66" y="20.32" smashed="yes">
+<instance part="X1" gate="-1" x="73.66" y="25.4" smashed="yes">
+<attribute name="NAME" x="73.66" y="26.289" size="1.778" layer="95" rot="R180"/>
+</instance>
+<instance part="X1" gate="-2" x="73.66" y="20.32" smashed="yes">
+<attribute name="VALUE" x="71.12" y="16.637" size="1.778" layer="96"/>
 <attribute name="NAME" x="73.66" y="21.209" size="1.778" layer="95" rot="R180"/>
-</instance>
-<instance part="X1" gate="-2" x="73.66" y="25.4" smashed="yes">
-<attribute name="VALUE" x="71.12" y="21.717" size="1.778" layer="96"/>
-<attribute name="NAME" x="73.66" y="26.289" size="1.778" layer="95" rot="R180"/>
 </instance>
 <instance part="GND1" gate="1" x="149.86" y="27.94" smashed="yes">
@@
 <pinref part="HLK1" gate="G$1" pin="AC1"/>
 <wire x1="86.36" y1="25.4" x2="88.9" y2="25.4" width="0.1524" layer="91"/>
-<wire x1="86.36" y1="25.4" x2="86.36" y2="-2.54" width="0.1524" layer="91"/>
+<pinref part="P+2" gate="VCC" pin="VCC"/>
+<pinref part="X1" gate="-1" pin="KL"/>
+<wire x1="78.74" y1="25.4" x2="86.36" y2="25.4" width="0.1524" layer="91"/>
 <junction x="86.36" y="25.4"/>
 <wire x1="86.36" y1="-2.54" x2="248.92" y2="-2.54" width="0.1524" layer="91"/>
@@
 <wire x1="238.76" y1="12.7" x2="248.92" y2="12.7" width="0.1524" layer="91"/>
 <junction x="248.92" y="12.7"/>
-<pinref part="P+2" gate="VCC" pin="VCC"/>
-<pinref part="X1" gate="-2" pin="KL"/>
-<wire x1="78.74" y1="25.4" x2="86.36" y2="25.4" width="0.1524" layer="91"/>
+<wire x1="86.36" y1="-2.54" x2="86.36" y2="25.4" width="0.1524" layer="91"/>
 </segment>
 </net>
@@
 <junction x="259.08" y="22.86"/>
 <wire x1="259.08" y1="-5.08" x2="83.82" y2="-5.08" width="0.1524" layer="91"/>
+<pinref part="GND2" gate="1" pin="0V"/>
+<junction x="259.08" y="-5.08"/>
+<pinref part="X1" gate="-2" pin="KL"/>
 <pinref part="HLK1" gate="G$1" pin="AC2"/>
+<wire x1="78.74" y1="20.32" x2="83.82" y2="20.32" width="0.1524" layer="91"/>
 <wire x1="83.82" y1="20.32" x2="88.9" y2="20.32" width="0.1524" layer="91"/>
 <wire x1="83.82" y1="-5.08" x2="83.82" y2="20.32" width="0.1524" layer="91"/>
-<pinref part="GND2" gate="1" pin="0V"/>
-<junction x="259.08" y="-5.08"/>
-<pinref part="X1" gate="-1" pin="KL"/>
-<wire x1="78.74" y1="20.32" x2="83.82" y2="20.32" width="0.1524" layer="91"/>
 <junction x="83.82" y="20.32"/>
 </segment>
@@
 </segment>
 </net>
-<net name="N$14" class="0">
-<segment>
-<pinref part="U$1" gate="G$1" pin="D1"/>
-<wire x1="157.48" y1="60.96" x2="127" y2="60.96" width="0.1524" layer="91"/>
-<pinref part="LED1" gate="G$1" pin="A"/>
-<wire x1="160.02" y1="76.2" x2="157.48" y2="76.2" width="0.1524" layer="91"/>
-<wire x1="157.48" y1="76.2" x2="157.48" y2="60.96" width="0.1524" layer="91"/>
-</segment>
-</net>
-<net name="N$15" class="0">
-<segment>
-<pinref part="U$1" gate="G$1" pin="D2"/>
-<wire x1="157.48" y1="58.42" x2="127" y2="58.42" width="0.1524" layer="91"/>
-<pinref part="LED2" gate="G$1" pin="A"/>
-<wire x1="162.56" y1="55.88" x2="157.48" y2="55.88" width="0.1524" layer="91"/>
-<wire x1="157.48" y1="55.88" x2="157.48" y2="58.42" width="0.1524" layer="91"/>
-</segment>
-</net>
 <net name="N$16" class="0">
 <segment>
-<pinref part="U$1" gate="G$1" pin="D3"/>
-<wire x1="127" y1="55.88" x2="154.94" y2="55.88" width="0.1524" layer="91"/>
-<wire x1="154.94" y1="55.88" x2="154.94" y2="35.56" width="0.1524" layer="91"/>
+<wire x1="83.82" y1="86.36" x2="83.82" y2="58.42" width="0.1524" layer="91"/>
+<wire x1="83.82" y1="86.36" x2="152.4" y2="86.36" width="0.1524" layer="91"/>
+<wire x1="152.4" y1="86.36" x2="152.4" y2="15.24" width="0.1524" layer="91"/>
+<pinref part="LED4" gate="G$1" pin="A"/>
+<wire x1="152.4" y1="15.24" x2="160.02" y2="15.24" width="0.1524" layer="91"/>
+<pinref part="U$1" gate="G$1" pin="D5"/>
+<wire x1="83.82" y1="58.42" x2="91.44" y2="58.42" width="0.1524" layer="91"/>
+</segment>
+</net>
+<net name="N$17" class="0">
+<segment>
+<wire x1="86.36" y1="83.82" x2="86.36" y2="60.96" width="0.1524" layer="91"/>
+<wire x1="86.36" y1="83.82" x2="154.94" y2="83.82" width="0.1524" layer="91"/>
+<wire x1="154.94" y1="83.82" x2="154.94" y2="35.56" width="0.1524" layer="91"/>
+<pinref part="LED3" gate="G$1" pin="A"/>
 <wire x1="154.94" y1="35.56" x2="160.02" y2="35.56" width="0.1524" layer="91"/>
-<pinref part="LED3" gate="G$1" pin="A"/>
-</segment>
-</net>
-<net name="N$17" class="0">
-<segment>
-<pinref part="U$1" gate="G$1" pin="D4"/>
-<wire x1="127" y1="53.34" x2="152.4" y2="53.34" width="0.1524" layer="91"/>
-<wire x1="152.4" y1="53.34" x2="152.4" y2="15.24" width="0.1524" layer="91"/>
-<wire x1="152.4" y1="15.24" x2="160.02" y2="15.24" width="0.1524" layer="91"/>
-<pinref part="LED4" gate="G$1" pin="A"/>
+<pinref part="U$1" gate="G$1" pin="D0"/>
+<wire x1="86.36" y1="60.96" x2="91.44" y2="60.96" width="0.1524" layer="91"/>
 </segment>
 </net>
@@
 </segment>
 </net>
+<net name="N$14" class="0">
+<segment>
+<pinref part="U$1" gate="G$1" pin="D2"/>
+<wire x1="127" y1="58.42" x2="157.48" y2="58.42" width="0.1524" layer="91"/>
+<wire x1="157.48" y1="58.42" x2="157.48" y2="55.88" width="0.1524" layer="91"/>
+<pinref part="LED2" gate="G$1" pin="A"/>
+<wire x1="157.48" y1="55.88" x2="162.56" y2="55.88" width="0.1524" layer="91"/>
+</segment>
+</net>
+<net name="N$15" class="0">
+<segment>
+<pinref part="U$1" gate="G$1" pin="D1"/>
+<pinref part="LED1" gate="G$1" pin="A"/>
+<wire x1="127" y1="60.96" x2="160.02" y2="60.96" width="0.1524" layer="91"/>
+<wire x1="160.02" y1="60.96" x2="160.02" y2="76.2" width="0.1524" layer="91"/>
+</segment>
+</net>

Commit message: refactoring
Parts:
- removed R1, R2, R3, R4: 1k, rcl:R-EU_0204/5
Connections:
- removed net N$10: R4.2, T4.B
- removed net N$17: LED3.A, U$1.D0
- removed net N$18: LED3.C, R3.1
- removed net N$20: LED1.C, R1.1
- net N$14: now also U$1.D5; no longer U$1.D2
- net N$15: now also U$1.D0; no longer U$1.D1
- net N$16: now also U$1.D7; no longer U$1.D5
- net N$19: now also LED3.A, U$1.D6; no longer LED2.C, R2.1
- net N$6: now also T4.B; no longer R4.1
- net N$7: now also LED3.C; no longer R3.2
- net N$8: now also LED2.C; no longer R2.2
- net N$9: now also LED1.C; no longer R1.2
Other:
- moved on the sheet: LED1, LED2, LED3, LED4, U$1

Commit message: refactoring
Parts:
- added C1, C2, C3, C4: (no value), rcl:CPOL-EUE5-5
- added C10, C11, C12, C5, C6, C7, C8, C9: (no value), rcl:C-EU025-024X044
- added IC1: PCF8574P, micro-philips:PCF8574P
- added OK1, OK2, OK3, OK4: PC814, optocoupler:PC814
- added R1, R10, R11, R12, R2, R3, R4, R5, R6, R7, R8, R9: (no value), rcl:R-EU_0204/5
- added X6: IN5, con-wago-500:W237-102
- added X7: IN6, con-wago-500:W237-102
Connections:
- new net N$10: C9.1, R4.2, R6.2
- new net N$17: IC1.SCL, U$1.D1
- new net N$18: IC1.SDA, U$1.D2
- new net N$20: C10.1, R3.2, R8.2
- new net N$21: C11.1, R10.2, R2.2
- new net N$22: C8.1, OK4.AC1, R1.1
- new net N$23: C11.2, R9.2, X7-1.KL
- new net N$24: C10.2, R7.2, X6-2.KL
- new net N$25: C9.2, R5.2, X6-1.KL
- new net N$26: R5.1, R6.1
- new net N$27: C12.1, C12.2, R1.2, R11.2, R12.2, X7-2.KL
- new net N$28: C7.1, OK3.AC1, R2.1
- new net N$29: C6.1, OK2.AC1, R3.1
- new net N$30: C5.1, OK1.AC1, R4.1
- new net N$31: R7.1, R8.1
- new net N$32: R10.1, R9.1
- new net N$33: R11.1, R12.1
- net 0V: now also C5.2, C6.2, C7.2, C8.2, OK1.AC2, OK2.AC2, OK3.AC2, OK4.AC2
- net GND: now also C1.-, C2.-, C3.-, C4.-, IC1.VSS, LED1.C, LED2.C, LED3.C, LED4.C, OK1.E, OK2.E, OK3.E, OK4.E
- net N$14: now also T2.B
- net N$15: now also T1.B
- net N$16: now also T4.B
- net N$19: now also T3.B
- net N$6: now also C1.+, IC1.P3, OK1.C; no longer LED4.C, T4.B
- net N$7: now also C2.+, IC1.P2, OK2.C; no longer LED3.C, T3.B
- net N$8: now also C3.+, IC1.P1, OK3.C; no longer LED2.C, T2.B
- net N$9: now also C4.+, IC1.P0, OK4.C; no longer LED1.C, T1.B
Other:
- moved on the sheet: LED1, LED2, LED3, LED4
